File: trigger_line.kicad_sch (KiCad schematic)
At the start: 2 parts, among them Q1 NTE3221, Q2 NTE3221

Commit message: schematic
Parts:
- removed Q1: NTE3221, NTE3221:DIP762W70P254L1990H508Q16N, symbol NTE3221:NTE3221
- removed Q2: NTE3221, DIP762W70P254L1990H508Q16N, symbol NTE3221:NTE3221
- added P1: 53048-0910, 53048-0910:53048-0910, symbol 53048-0910:53048-0910
- added P2: 53048-1010, 53048-1010:53048-1010, symbol 53048-1010:53048-1010
- added R1, R2, R3, R4, R5, R6, R7, R8: 270, symbol Device:R
- added R10, R11, R12, R13, R14, R15, R16, R9: 390, symbol Device:R
- added U1, U2: ILQ30, ILQ30:DIP762W51P254L1992H425Q16, symbol ILQ30:ILQ30
Connections:
- new net: P1.3, R3.1
- new net: R3.2, U1.5
- new net: P2.8, R16.2, U2.9
- new net: R5.2, U2.1
- new net: P2.7, R15.1, U2.12
- new net: P2.6, R14.2, U2.13
- new net: P2.5, R13.1, U2.16
- new net: R6.2, U2.4
- new net: R7.2, U2.5
- new net: R8.2, U2.8
- new net: P2.1, R9.1, U1.16
- new net: P2.2, R10.2, U1.13
- new net: P2.3, R11.1, U1.12
- new net: P2.4, R12.2, U1.9
- new net: R1.2, U1.1
- new net: R2.2, U1.4
- new net: R4.2, U1.8
- new net: P1.6, R6.1
- new net: P1.1, R1.1
- new net: P1.2, R2.1
- new net: P1.4, R4.1
- new net: P1.5, R5.1
- new net: P1.7, R7.1
- new net: P1.8, R8.1
- new net +5V: P2.9, U1.10, U1.11, U1.14, U1.15, U2.10, U2.11, U2.14, U2.15
- new net GND: P1.9, P2.10, R10.1, R11.2, R12.1, R13.2, R14.1, R15.2, R16.1, R9.2, U1.2, U1.3, U1.6, U1.7, U2.2, U2.3, U2.6, U2.7

Commit message: first order
Parts:
- removed R1, R2, R3, R4, R5, R6, R7, R8: 270, symbol Device:R
- removed R10, R11, R12, R13, R14, R15, R16, R9: 390, symbol Device:R
- added R1, R2, R3, R4, R5, R6, R7, R8: RNMF14FTC270R, STA_RNMF14_STP, symbol 2024-01-01_18-12-41:RNMF14FTC270R
- added R10, R11, R12, R13, R14, R15, R16, R9: RNMF14FTC390R, STA_RNMF14_STP, symbol 2024-01-01_18-12-10:RNMF14FTC390R
Connections:
- net GND: now also R10.2, R11.2, R12.2, R13.2, R14.2, R15.2, R16.2, R9.2; no longer P1.9, U1.2, U1.3, U1.6, U1.7, U2.2, U2.3, U2.6, U2.7
- net at P1.3: now also R3.1
- net at U1.5: now also R3.2
- net at P2.8, U2.9: now also R16.1
- net at U2.1: now also R5.2
- net at P2.7, U2.12: now also R15.1
- net at P2.6, U2.13: now also R14.1
- net at P2.5, U2.16: now also R13.1
- net at U2.4: now also R6.2
- net at U2.5: now also R7.2
- net at U2.8: now also R8.2
- net at P2.1, U1.16: now also R9.1
- net at P2.2, U1.13: now also R10.1
- net at P2.3, U1.12: now also R11.1
- net at P2.4, U1.9: now also R12.1
- net at U1.1: now also R1.2
- net at U1.4: now also R2.2
- net at U1.8: now also R4.2
- net at P1.6: now also R6.1
- net at P1.1: now also R1.1
- net at P1.2: now also R2.1
- net at P1.4: now also R4.1
- net at P1.5: now also R5.1
- net at P1.7: now also R7.1
- net at P1.8: now also R8.1
- new net GNDA: P1.9, U1.2, U1.3, U1.6, U1.7, U2.2, U2.3, U2.6, U2.7
Other:
- moved on the sheet: P1, P2, U1, U2
